File: Hardware/Teensy_3_1 XBee Adapter.brd (EAGLE design)
At the start: 33 x 86.4 mm, 35 parts

Commit message: Final proto fixes
Parts:
- removed SJ2: D_TX, SparkFun-Passives:PAD-JUMPER-2-NC_BY_PASTE_YES_SILK
- added LOGO1: SFE_LOGO_FLAME.2_INCH, SparkFun-Aesthetics:SFE_LOGO_FLAME_.2
- moved FRAME1 97.7 mm to (68.6, 34.3)
Connections:
- removed net AGND: JP1.AGND, JP7.3, SJ2.1
- net GND: now also JP1.AGND, JP7.3; no longer SJ2.2
Routing:
- net AGND: track 15.7 -> 0.00 mm, vias 1 -> 0
- net GND: track 38.9 -> 49.9 mm
- net XBEE_VDD: track 61.1 -> 62.2 mm
Other:
- board text added: "3.1"
- board text added: "Teensy"
- board text added: "Units in inches"
- board text added: "v10"
- board text removed: "AGND"
- board text removed: "DGND"
- board text removed: "Teensy 3.1"
- board text removed: "v03"
