File: Hardware/Teensy_3_1 XBee Adapter.sch (EAGLE design)
At the start: 35 parts

Commit message: removed micro fids, added regular 1x2
Parts:
- FID1, FID2: value FIDUCIALUFIDUCIAL -> FIDUCIAL1X2; device SparkFun-Aesthetics:FIDUCIALUFIDUCIAL -> SparkFun-Aesthetics:FIDUCIAL1X2
Changed lines of the file:
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@@
 <?xml version="1.0" encoding="utf-8"?>
 <!DOCTYPE eagle SYSTEM "eagle.dtd">
-<eagle version="7.1.0">
+<eagle version="7.2.0">
 <drawing>
 <settings>
@@
 <part name="R2" library="SparkFun-Resistors" deviceset="1KOHM1/10W1%(0603)" device="" value="1k"/>
 <part name="GND12" library="SparkFun" deviceset="GND" device=""/>
-<part name="FID1" library="SparkFun-Aesthetics" deviceset="FIDUCIAL" device="UFIDUCIAL" value="FIDUCIALUFIDUCIAL"/>
-<part name="FID2" library="SparkFun-Aesthetics" deviceset="FIDUCIAL" device="UFIDUCIAL" value="FIDUCIALUFIDUCIAL"/>
 <part name="STANDOFF1" library="SparkFun-Electromechanical" deviceset="STAND-OFF" device=""/>
 <part name="STANDOFF2" library="SparkFun-Electromechanical" deviceset="STAND-OFF" device=""/>
@@
 <part name="JP8" library="SparkFun-Connectors" deviceset="M02" device="PTH" value="DNP"/>
 <part name="LOGO1" library="SparkFun-Aesthetics" deviceset="SFE_LOGO_FLAME" device=".2_INCH"/>
+<part name="FID1" library="SparkFun-Aesthetics" deviceset="FIDUCIAL" device="1X2"/>
+<part name="FID2" library="SparkFun-Aesthetics" deviceset="FIDUCIAL" device="1X2"/>
 </parts>
 <sheets>
@@
 <instance part="R2" gate="G$1" x="73.66" y="152.4" rot="R90"/>
 <instance part="GND12" gate="1" x="73.66" y="132.08"/>
-<instance part="FID1" gate="G$1" x="228.6" y="27.94"/>
-<instance part="FID2" gate="G$1" x="233.68" y="27.94"/>
 <instance part="STANDOFF1" gate="G$1" x="238.76" y="27.94"/>
 <instance part="STANDOFF2" gate="G$1" x="243.84" y="27.94"/>
@@
 <instance part="JP8" gate="G$1" x="96.52" y="76.2" rot="R180"/>
 <instance part="LOGO1" gate="G$1" x="129.54" y="27.94"/>
+<instance part="FID1" gate="G$1" x="233.68" y="27.94"/>
+<instance part="FID2" gate="G$1" x="228.6" y="27.94"/>
 </instances>
 <busses>
